File: PCB/Mini/hre-clone.kicad_sch (KiCad schematic)
At the start: 23 parts, among them SW1 SW_DIP_x04, U1 74LS258, U10 MC6845, U11 MC6845, U12 DIL14, U13 7402, U2 74LS174, U3 74LS257, U4 74LS244, U5 2716, U6 2716, U7 74LS05, U8 74LS155, U9 74LS257

Commit message: Even more Mini!
Shuffled some chips and traces, added beveled corners and made the text labelling more normal.
Parts:
- removed R1, R2, R3, R4: R, Resistor_THT:R_Axial_DIN0309_L9.0mm_D3.2mm_P12.70mm_Horizontal, symbol Device:R
- added RN1: 3300 ohm, Resistor_THT:R_Array_SIP5, symbol Device:R_Network04_US
- R5: value R -> 3300
Connections:
- net DIP1: now also RN1.2 (R1)
- net DIP2: now also RN1.3 (R2)
- net DIP3: now also RN1.4 (R3)
- net DIP4: now also RN1.5 (R4)
- net VCC: now also RN1.1 (common)
Other:
- moved on the sheet: SW1
